File: 2floor_for_orange_pi.kicad_sch (KiCad schematic)
At the start: 10 parts, among them J1 Orange_PI_PC_ONE_40Pin_Header, J2 I2S1 DAC Socket, J3 I2S2 ADC Socket, J4 +3V3 Header, J5 +5V Header, J6 GND Header, J7 STM32 DEBUG Header, J8 OPI Conn Debug Socket, J9 OPI Conn Debug Header

Commit message: completed 1st tracing
Parts:
- added J11: OPI SPI0 Header, Connector_PinHeader_2.54mm:PinHeader_1x04_P2.54mm_Vertical, symbol PCM_SL_Pin_Headers:PINHD_1x4_Male
- added J12: ST7735 Header, Connector_PinHeader_2.54mm:PinHeader_1x05_P2.54mm_Vertical, symbol PCM_SL_Pin_Headers:PINHD_1x5_Male
- added J13, J14, J15, J16: SPI5 Header, Connector_PinHeader_2.54mm:PinHeader_1x05_P2.54mm_Vertical, symbol PCM_SL_Pin_Headers:PINHD_1x5_Male
- added J17: STM32 GPIO Header, Connector_PinHeader_2.54mm:PinHeader_1x03_P2.54mm_Vertical, symbol PCM_SL_Pin_Headers:PINHD_1x3_Male
Connections:
- net GND: now also J13.5, J14.5, J15.5, J16.5
- net SPI5_MISO: now also J13.3, J14.3, J15.3, J16.3
- net SPI5_MOSI: now also J13.2, J14.2, J15.2, J16.2
- net SPI5_SCK: now also J13.1, J14.1, J15.1, J16.1
- net SPI5_CS1: now reaches U1.15 (B1)
- net SPI5_CS1: now also J14.4
- net ST7735_RES: now reaches U1.16 (B2)
- net ST7735_RES: now also J12.5
- net ST7735_CS: now reaches U1.17 (B10)
- net ST7735_CS: now also J12.4, J13.4
- net ST7735_DC: now reaches U1.23 (B14)
- net ST7735_DC: now also J12.3
- net ST7735_BL: now reaches U1.25 (A8)
- net ST7735_BL: now also J12.2
- net SPI5_CS2: now reaches U1.26 (A9)
- net SPI5_CS2: now also J15.4
- net TIM1_PWM_OUTPUT: now reaches U1.28 (A11)
- net TIM1_PWM_OUTPUT: now also J12.1
- net at U1.3 (C14): now also J17.1
- net SPI5_CS3: now reaches U1.36 (B8)
- net SPI5_CS3: now also J16.4
- net at U1.37 (B9): now also J17.3
- net at U1.4 (C15): now also J17.2
- net at J1.19 ((PC0)/SPI0_MOSI): now also J11.2
- net at J1.21 ((PC1)/SPI0_MISO): now also J11.3
- net at J1.23 ((PC2)/SPI0_SCK): now also J11.1
- net at J1.24 ((PC3}/SPI0_CS): now also J11.4
- no-connect marks 2 -> 5
Other:
- moved on the sheet: J4, J5, J6
