File: 2floor_for_orange_pi.kicad_pcb (KiCad board)
At the start: 2 copper layers, 56 x 68 mm, 10 parts, among them J1 Orange_PI_PC_ONE_40Pin_Header, J2 I2S1 DAC Socket, J3 I2S2 ADC Socket, J4 +3V3 Header, J5 +5V Header, J6 GND Header, J7 STM32 DEBUG Header, J8 OPI Conn Debug Socket, J9 OPI Conn Debug Header

Commit message: completed 1st tracing
Parts:
- added J11: OPI SPI0 Header, Connector_PinHeader_2.54mm:PinHeader_1x04_P2.54mm_Vertical, B.Cu at (49.7, 63.1)
- added J12: ST7735 Header, Connector_PinHeader_2.54mm:PinHeader_1x05_P2.54mm_Vertical, B.Cu at (48.7, 22.2)
- added J13: SPI5 Header, Connector_PinHeader_2.54mm:PinHeader_1x05_P2.54mm_Vertical, B.Cu at (52.3, 19.7)
- added J14: SPI5 Header, Connector_PinHeader_2.54mm:PinHeader_1x05_P2.54mm_Vertical, B.Cu at (56.0, 19.7)
- added J15: SPI5 Header, Connector_PinHeader_2.54mm:PinHeader_1x05_P2.54mm_Vertical, B.Cu at (59.6, 19.7)
- added J16: SPI5 Header, Connector_PinHeader_2.54mm:PinHeader_1x05_P2.54mm_Vertical, B.Cu at (63.2, 19.7)
- added J17: STM32 GPIO Header, Connector_PinHeader_2.54mm:PinHeader_1x03_P2.54mm_Vertical, B.Cu at (30.5, 19.4)
- moved J6 7.23 mm to (67.3, 22.2)
- moved J8 7.23 mm to (74.5, 39.3)
- moved J1 7.23 mm to (25.4, 23.9)
- moved U1 7.23 mm to (36.6, 48.0)
- moved J2 7.23 mm to (74.6, 49.8)
- moved J4 7.23 mm to (74.5, 22.2)
- moved J5 7.23 mm to (70.9, 22.2)
- moved J9 7.23 mm to (70.7, 39.3)
- moved J7 7.09 mm to (48.9, 39.2)
- moved J3 5.63 mm to (74.6, 68.7)
Connections:
- J1 pad 19: unconnected-(J1-(PC0)/SPI0_MOSI-Pad19) -> Net-(J1-(PC0)/SPI0_MOSI)
- J1 pad 21: unconnected-(J1-(PC1)/SPI0_MISO-Pad21) -> Net-(J1-(PC1)/SPI0_MISO)
- J1 pad 23: unconnected-(J1-(PC2)/SPI0_SCK-Pad23) -> Net-(J1-(PC2)/SPI0_SCK)
- J1 pad 24: unconnected-(J1-(PC3}/SPI0_CS-Pad24) -> Net-(J1-(PC3}/SPI0_CS)
- U1 pad 15: unconnected-(U1-B1-Pad15) -> /SPI5_CS1
- U1 pad 16: unconnected-(U1-B2-Pad16) -> /ST7735_RES
- U1 pad 17: unconnected-(U1-B10-Pad17) -> /ST7735_CS
- U1 pad 23: unconnected-(U1-B14-Pad23) -> /ST7735_DC
- U1 pad 25: unconnected-(U1-A8-Pad25) -> /ST7735_BL
- U1 pad 26: unconnected-(U1-A9-Pad26) -> /SPI5_CS2
- U1 pad 28: unconnected-(U1-A11-Pad28) -> /TIM1_PWM_OUTPUT
- U1 pad 3: unconnected-(U1-C14-Pad3) -> Net-(U1-C14)
- U1 pad 36: unconnected-(U1-B8-Pad36) -> /SPI5_CS3
- U1 pad 37: unconnected-(U1-B9-Pad37) -> Net-(U1-B9)
- U1 pad 4: unconnected-(U1-C15-Pad4) -> Net-(U1-C15)
Routing:
- net GND: track 0.00 -> 273.1 mm, vias 0 -> 15
- net +5V: track 0.00 -> 180.5 mm, vias 0 -> 4
- net +3V3: track 0.00 -> 179.1 mm, vias 0 -> 10
- net /SPI5_MOSI: track 0.00 -> 69.1 mm, vias 0 -> 5
- net /ST7735_BL: track 0.00 -> 62.4 mm, vias 0 -> 3
- net /SPI5_CS2: track 0.00 -> 61.7 mm, vias 0 -> 4
- net /I2S2_SCK: track 0.00 -> 61.7 mm, vias 0 -> 5
- net /SPI5_SCK: track 0.00 -> 56.2 mm, vias 0 -> 1
- net /ST7735_DC: track 0.00 -> 54.0 mm, vias 0 -> 5
- net /ST7735_CS: track 0.00 -> 52.8 mm, vias 0 -> 2
- net /I2S2_DATA_IN: track 0.00 -> 52.5 mm, vias 0 -> 2
- net /SPI5_CS3: track 0.00 -> 52.3 mm, vias 0 -> 4
- net /SPI5_MISO: track 0.00 -> 51.7 mm, vias 0 -> 2
- net /I2S2_BCK: track 0.00 -> 50.6 mm, vias 0 -> 2
- net /TIM1_PWM_OUTPUT: track 0.00 -> 50.3 mm, vias 0 -> 3
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- added copper zone on B.Cu, net GND
Other:
- board size 56 x 68 mm -> 56.5 x 69.9 mm
- board text added: "2023-2024 (c) AxelRouse dev@1cdev.ru boards@1cdev.ru O!BLT Shield"
- board text added: "https://github.com/alexeyavb/Orangeblock.git"

Commit message: sended to print
Routing:
- net GND: track 273.1 -> 275.9 mm, vias 15 -> 14
Changed lines of the file:
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@@
 		)
 		(fp_text user "${REFERENCE}"
-			(at 0 -2.54 360)
+			(at 0 -2.54 0)
 			(layer "B.Fab")
 			(effects
@@
 	)
 	(segment
+		(start 55.98 29.84)
+		(end 57.36 29.84)
+		(width 0.8)
+		(layer "F.Cu")
+		(net 3)
+	)
+	(segment
 		(start 24.21 35.59)
 		(end 24.21 37.85)
@@
 	)
 	(segment
+		(start 57.36 29.84)
+		(end 59.49 31.97)
+		(width 0.8)
+		(layer "F.Cu")
+		(net 3)
+	)
+	(segment
 		(start 72.29 48.25)
 		(end 72.1 48.25)
@@
 	)
 	(segment
-		(start 51.19 28.74)
-		(end 51.24 28.74)
-		(width 0.4)
-		(layer "F.Cu")
-		(net 3)
-	)
-	(segment
 		(start 22.89 29.01)
 		(end 21.62 29.01)
@@
 	)
 	(segment
-		(start 51.24 28.74)
-		(end 52.34 29.84)
-		(width 0.4)
-		(layer "F.Cu")
-		(net 3)
-	)
-	(segment
 		(start 63.22 31.61)
 		(end 63.22 29.84)
@@
 		(size 0.6)
 		(drill 0.3)
-		(layers "F.Cu" "B.Cu")
-		(net 3)
-	)
-	(via
-		(at 51.19 28.74)
-		(size 0.6)
-		(drill 0.3)
